File: Macropad V2.kicad_pcb (KiCad board)
At the start: 2 copper layers, 57.2 x 82 mm, 20 parts, among them SW1 SW_Push, SW2 SW_Push, SW3 SW_Push, SW4 SW_Push, SW5 SW_Push, SW6 SW_Push, SW7 SW_Push, SW8 SW_Push, SW9 SW_Push, U1 MOUDLE-SEEEDUINO-XIAO

Commit message: art
Other:
- board text added: "A tribute to the Macropad that started it all :)"
Changed lines of the file:
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@@
 		(embedded_fonts no)
+	)
+	(gr_arc
+		(start 110.39 68.72)
+		(mid 111.717999 66.439402)
+		(end 114.062754 65.228272)
+		(stroke
+			(width 0.1)
+			(type default)
+		)
+		(layer "B.SilkS")
 	)
 	(gr_rect
@@
 		)
 	)
+	(gr_text "A tribute to the Macropad that started it all :)"
+		(at 126.63 75.97 315)
+		(layer "B.SilkS")
+		(effects
+			(font
+				(size 1 1)
+				(thickness 0.1)
+			)
+			(justify left bottom mirror)
+		)
+	)
